Commit message: remove unused resources

File: urdf/H6.urdf (robot description, URDF)
Before this commit: robot H6_robot, 22 links, 21 joints
Links:
- link LAnklePitch: geometry collision mesh filename=meshes/LAnklePitch_0.10.stl scale=0.1 0.1 0.1; visual mesh filename=meshes/LAnklePitch_0.10.stl scale=0.1 0.1 0.1
- link LAnkleRoll: geometry collision mesh filename=meshes/LAnkleRoll_0.10.stl scale=0.1 0.1 0.1; visual mesh filename=meshes/LAnkleRoll_0.10.stl scale=0.1 0.1 0.1
- link LBicep: geometry collision mesh filename=meshes/LShoulderRoll_0.10.stl scale=0.1 0.1 0.1; visual mesh filename=meshes/LShoulderRoll_0.10.stl scale=0.1 0.1 0.1
- link LElbow: geometry collision mesh filename=meshes/LElbow_0.10.stl scale=0.1 0.1 0.1; visual mesh filename=meshes/LElbow_0.10.stl scale=0.1 0.1 0.1
- link LHipPitch: geometry collision mesh filename=meshes/LHipPitch_0.10.stl scale=0.1 0.1 0.1; visual mesh filename=meshes/LHipPitch_0.10.stl scale=0.1 0.1 0.1
- link LHipRoll: geometry collision mesh filename=meshes/LHipRoll_0.10.stl scale=0.1 0.1 0.1; visual mesh filename=meshes/LHipRoll_0.10.stl scale=0.1 0.1 0.1
- link LHipYaw: geometry collision mesh filename=meshes/LHipYaw_0.10.stl scale=0.1 0.1 0.1; visual mesh filename=meshes/LHipYaw_0.10.stl scale=0.1 0.1 0.1
- link LKnee: geometry collision mesh filename=meshes/LKnee_0.10.stl scale=0.1 0.1 0.1; visual mesh filename=meshes/LKnee_0.10.stl scale=0.1 0.1 0.1
- link LShoulder: geometry collision mesh filename=meshes/LShoulderPitch_0.10.stl scale=0.1 0.1 0.1; visual mesh filename=meshes/LShoulderPitch_0.10.stl scale=0.1 0.1 0.1
- link RAnklePitch: geometry collision mesh filename=meshes/RAnklePitch_0.10.stl scale=0.1 0.1 0.1; visual mesh filename=meshes/RAnklePitch_0.10.stl scale=0.1 0.1 0.1
- link RAnkleRoll: geometry collision mesh filename=meshes/RAnkleRoll_0.10.stl scale=0.1 0.1 0.1; visual mesh filename=meshes/RAnkleRoll_0.10.stl scale=0.1 0.1 0.1
- link RBicep: geometry collision mesh filename=meshes/RShoulderRoll_0.10.stl scale=0.1 0.1 0.1; visual mesh filename=meshes/RShoulderRoll_0.10.stl scale=0.1 0.1 0.1
- link RElbow: geometry collision mesh filename=meshes/RElbow_0.10.stl scale=0.1 0.1 0.1; visual mesh filename=meshes/RElbow_0.10.stl scale=0.1 0.1 0.1
- link RHipPitch: geometry collision mesh filename=meshes/RHipPitch_0.10.stl scale=0.1 0.1 0.1; visual mesh filename=meshes/RHipPitch_0.10.stl scale=0.1 0.1 0.1
- link RHipRoll: geometry collision mesh filename=meshes/RHipRoll_0.10.stl scale=0.1 0.1 0.1; visual mesh filename=meshes/RHipRoll_0.10.stl scale=0.1 0.1 0.1
- link RHipYaw: geometry collision mesh filename=meshes/RHipYaw_0.10.stl scale=0.1 0.1 0.1; visual mesh filename=meshes/RHipYaw_0.10.stl scale=0.1 0.1 0.1
- link RKnee: geometry collision mesh filename=meshes/RKnee_0.10.stl scale=0.1 0.1 0.1; visual mesh filename=meshes/RKnee_0.10.stl scale=0.1 0.1 0.1
- link RShoulder: geometry collision mesh filename=meshes/RShoulderPitch_0.10.stl scale=0.1 0.1 0.1; visual mesh filename=meshes/RShoulderPitch_0.10.stl scale=0.1 0.1 0.1
- link head: geometry collision mesh filename=meshes/Head_0.10.stl scale=0.1 0.1 0.1; visual mesh filename=meshes/Head_0.10.stl scale=0.1 0.1 0.1
- link neck: geometry collision mesh filename=meshes/Neck_0.10.stl scale=0.1 0.1 0.1; visual mesh filename=meshes/Neck_0.10.stl scale=0.1 0.1 0.1
- link torso: geometry collision mesh filename=meshes/Torso_0.10.stl scale=0.1 0.1 0.1; visual mesh filename=meshes/Torso_0.10.stl scale=0.1 0.1 0.1
Joints:
- joint LAnklePitch: origin xyz=0.0 -0.065 -0.003 rpy=0.0 0.0 0.0 -> xyz=0.0 -0.065 -0.008 rpy=0.0 0.0 0.0
- joint LAnkleRoll: origin xyz=0.0 -0.036 0.0 rpy=0.0 0.0 0.0 -> xyz=0.0 -0.035 0.0 rpy=0.0 0.0 0.0
- joint LElbowYaw: limit lower=-1.5757 upper=0.31415 effort=1.329 velocity=8.26797 -> lower=-1.5757 upper=1.5757 effort=1.329 velocity=8.26797; origin xyz=0.0745 0.0 0.0 rpy=0 -1.5757 0 -> xyz=0.075 0.0 0.0 rpy=0 -1.5757 0
- joint LHipPitch: origin xyz=0.0 -0.0426 0.0 rpy=0.0 0.0 0.0 -> xyz=0.0 -0.044 0.0 rpy=0.0 0.0 0.0
- joint LHipRoll: origin xyz=0.0 0.0 0.0905 rpy=1.5757 3.14159 0.0 -> xyz=0.0 0.0 0.09 rpy=1.5757 3.14159 0.0
- joint LHipYaw: origin xyz=0.036 -0.035 0.0 rpy=-1.5757 0.0 3.14159 -> xyz=0.035 -0.035 0.0 rpy=-1.5757 0.0 3.14159
- joint LKnee: limit lower=0.0 upper=2.05 effort=1.329 velocity=8.26797 -> lower=0.0 upper=1.5757 effort=1.329 velocity=8.26797; origin xyz=0.0 -0.065 -0.003 rpy=0.0 0.0 0.0 -> xyz=0.0 -0.06 0.0 rpy=0.0 0.0 0.0
- joint LShoulderPitch: origin xyz=0.05 0.0 0.005 rpy=0 0 0 -> xyz=0.05 0.0 0.006 rpy=0 0 0
- joint LShoulderRoll: origin xyz=0.041 0.0 0.0 rpy=0 0 0 -> xyz=0.04 0.0 0.0 rpy=0 0 0
- joint RAnklePitch: origin xyz=0.0 -0.065 -0.003 rpy=0.0 0.0 0.0 -> xyz=0.0 -0.065 -0.008 rpy=0.0 0.0 0.0
- joint RAnkleRoll: origin xyz=0.0 -0.036 0.0 rpy=0.0 0.0 0.0 -> xyz=0.0 -0.035 0.0 rpy=0.0 0.0 0.0
- joint RElbowYaw: limit lower=-0.31415 upper=1.5757 effort=1.329 velocity=8.26797 -> lower=-1.5757 upper=1.5757 effort=1.329 velocity=8.26797; origin xyz=-0.0745 0.0 0.0 rpy=0 -1.575 3.14159 -> xyz=-0.075 0.0 0.0 rpy=0 -1.575 3.14159
- joint RHipPitch: origin xyz=0.0 -0.0426 0.0 rpy=0.0 0.0 0.0 -> xyz=0.0 -0.044 0.0 rpy=0.0 0.0 0.0
- joint RHipRoll: origin xyz=0.0 0.0 0.0905 rpy=1.5757 3.14159 0.0 -> xyz=0.0 0.0 0.09 rpy=1.5757 3.14159 0.0
- joint RHipYaw: origin xyz=-0.036 -0.035 0.0 rpy=-1.5757 0.0 3.14159 -> xyz=-0.035 -0.035 0.0 rpy=-1.5757 0.0 3.14159
- joint RKnee: limit lower=0.0 upper=2.05 effort=1.329 velocity=8.26797 -> lower=0.0 upper=1.5757 effort=1.329 velocity=8.26797; origin xyz=0.0 -0.065 -0.003 rpy=0.0 0.0 0.0 -> xyz=0.0 -0.06 0.0 rpy=0.0 0.0 0.0
- joint RShoulderPitch: origin xyz=-0.05 0.0 0.005 rpy=0 0 0 -> xyz=-0.05 0.0 0.006 rpy=0 0 0
- joint RShoulderRoll: origin xyz=-0.041 0.0 0.0 rpy=0 0 0 -> xyz=-0.04 0.0 0.0 rpy=0 0 0
- joint head_to_neck: origin xyz=0.0 0.0 0.0 rpy=0 0 -3.1415 -> xyz=0.0 -0.0 0.0 rpy=0 0 -3.1415
- joint neck_to_torso: origin xyz=0.0 0.0466 0.0053 rpy=0 0 0 -> xyz=0.0 0.045 0.006 rpy=0 0 0
