Commit message: modify mesh path

File: H6.urdf (robot description, URDF)
Before this commit: robot H6_robot, 22 links, 21 joints
Links:
- link LAnklePitch: geometry collision mesh filename=meshes/LAnklePitch_0.10.stl scale=0.1 0.1 0.1; visual mesh filename=meshes/LAnklePitch_0.10.stl scale=0.1 0.1 0.1
- link LAnkleRoll: geometry collision mesh filename=meshes/LAnkleRoll_0.10.stl scale=0.1 0.1 0.1; visual mesh filename=meshes/LAnkleRoll_0.10.stl scale=0.1 0.1 0.1
- link LBicep: geometry collision mesh filename=meshes/LShoulderRoll_0.10.stl scale=0.1 0.1 0.1; visual mesh filename=meshes/LShoulderRoll_0.10.stl scale=0.1 0.1 0.1
- link LElbow: geometry collision mesh filename=meshes/LElbow_0.10.stl scale=0.1 0.1 0.1; visual mesh filename=meshes/LElbow_0.10.stl scale=0.1 0.1 0.1
- link LHipPitch: geometry collision mesh filename=meshes/LHipPitch_0.10.stl scale=0.1 0.1 0.1; visual mesh filename=meshes/LHipPitch_0.10.stl scale=0.1 0.1 0.1
- link LHipRoll: geometry collision mesh filename=meshes/LHipRoll_0.10.stl scale=0.1 0.1 0.1; visual mesh filename=meshes/LHipRoll_0.10.stl scale=0.1 0.1 0.1
- link LHipYaw: geometry collision mesh filename=meshes/LHipYaw_0.10.stl scale=0.1 0.1 0.1; visual mesh filename=meshes/LHipYaw_0.10.stl scale=0.1 0.1 0.1
- link LKnee: geometry collision mesh filename=meshes/LKnee_0.10.stl scale=0.1 0.1 0.1; visual mesh filename=meshes/LKnee_0.10.stl scale=0.1 0.1 0.1
- link LShoulder: geometry collision mesh filename=meshes/LShoulderPitch_0.10.stl scale=0.1 0.1 0.1; visual mesh filename=meshes/LShoulderPitch_0.10.stl scale=0.1 0.1 0.1
- link RAnklePitch: geometry collision mesh filename=meshes/RAnklePitch_0.10.stl scale=0.1 0.1 0.1; visual mesh filename=meshes/RAnklePitch_0.10.stl scale=0.1 0.1 0.1
- link RAnkleRoll: geometry collision mesh filename=meshes/RAnkleRoll_0.10.stl scale=0.1 0.1 0.1; visual mesh filename=meshes/RAnkleRoll_0.10.stl scale=0.1 0.1 0.1
- link RBicep: geometry collision mesh filename=meshes/RShoulderRoll_0.10.stl scale=0.1 0.1 0.1; visual mesh filename=meshes/RShoulderRoll_0.10.stl scale=0.1 0.1 0.1
- link RElbow: geometry collision mesh filename=meshes/RElbow_0.10.stl scale=0.1 0.1 0.1; visual mesh filename=meshes/RElbow_0.10.stl scale=0.1 0.1 0.1
- link RHipPitch: geometry collision mesh filename=meshes/RHipPitch_0.10.stl scale=0.1 0.1 0.1; visual mesh filename=meshes/RHipPitch_0.10.stl scale=0.1 0.1 0.1
- link RHipRoll: geometry collision mesh filename=meshes/RHipRoll_0.10.stl scale=0.1 0.1 0.1; visual mesh filename=meshes/RHipRoll_0.10.stl scale=0.1 0.1 0.1
- link RHipYaw: geometry collision mesh filename=meshes/RHipYaw_0.10.stl scale=0.1 0.1 0.1; visual mesh filename=meshes/RHipYaw_0.10.stl scale=0.1 0.1 0.1
- link RKnee: geometry collision mesh filename=meshes/RKnee_0.10.stl scale=0.1 0.1 0.1; visual mesh filename=meshes/RKnee_0.10.stl scale=0.1 0.1 0.1
- link RShoulder: geometry collision mesh filename=meshes/RShoulderPitch_0.10.stl scale=0.1 0.1 0.1; visual mesh filename=meshes/RShoulderPitch_0.10.stl scale=0.1 0.1 0.1
- link head: geometry collision mesh filename=meshes/Head_0.10.stl scale=0.1 0.1 0.1; visual mesh filename=meshes/Head_0.10.stl scale=0.1 0.1 0.1
- link neck: geometry collision mesh filename=meshes/Neck_0.10.stl scale=0.1 0.1 0.1; visual mesh filename=meshes/Neck_0.10.stl scale=0.1 0.1 0.1
- link torso: geometry collision mesh filename=meshes/Torso_0.10.stl scale=0.1 0.1 0.1; visual mesh filename=meshes/Torso_0.10.stl scale=0.1 0.1 0.1

Commit message: commit H5.urdf

File: H6.urdf (robot description, URDF)
Before this commit: robot H6_robot, 22 links, 21 joints
Links:
- removed link base_link
- link LAnklePitch: geometry collision mesh filename=meshes/LAnklePitch_0.10.stl scale=0.1 0.1 0.1; visual mesh filename=meshes/LAnklePitch_0.10.stl scale=0.1 0.1 0.1
- link LAnkleRoll: geometry collision mesh filename=meshes/LAnkleRoll_0.10.stl scale=0.1 0.1 0.1; visual mesh filename=meshes/LAnkleRoll_0.10.stl scale=0.1 0.1 0.1
- link LBicep: geometry collision mesh filename=meshes/LShoulderRoll_0.10.stl scale=0.1 0.1 0.1; visual mesh filename=meshes/LShoulderRoll_0.10.stl scale=0.1 0.1 0.1
- link LElbow: geometry collision mesh filename=meshes/LElbow_0.10.stl scale=0.1 0.1 0.1; visual mesh filename=meshes/LElbow_0.10.stl scale=0.1 0.1 0.1
- link LHipPitch: geometry collision mesh filename=meshes/LHipPitch_0.10.stl scale=0.1 0.1 0.1; visual mesh filename=meshes/LHipPitch_0.10.stl scale=0.1 0.1 0.1
- link LHipRoll: geometry collision mesh filename=meshes/LHipRoll_0.10.stl scale=0.1 0.1 0.1; visual mesh filename=meshes/LHipRoll_0.10.stl scale=0.1 0.1 0.1
- link LHipYaw: geometry collision mesh filename=meshes/LHipYaw_0.10.stl scale=0.1 0.1 0.1; visual mesh filename=meshes/LHipYaw_0.10.stl scale=0.1 0.1 0.1
- link LKnee: geometry collision mesh filename=meshes/LKnee_0.10.stl scale=0.1 0.1 0.1; visual mesh filename=meshes/LKnee_0.10.stl scale=0.1 0.1 0.1
- link LShoulder: geometry collision mesh filename=meshes/LShoulderPitch_0.10.stl scale=0.1 0.1 0.1; visual mesh filename=meshes/LShoulderPitch_0.10.stl scale=0.1 0.1 0.1
- link RAnklePitch: geometry collision mesh filename=meshes/RAnklePitch_0.10.stl scale=0.1 0.1 0.1; visual mesh filename=meshes/RAnklePitch_0.10.stl scale=0.1 0.1 0.1
- link RAnkleRoll: geometry collision mesh filename=meshes/RAnkleRoll_0.10.stl scale=0.1 0.1 0.1; visual mesh filename=meshes/RAnkleRoll_0.10.stl scale=0.1 0.1 0.1
- link RBicep: geometry collision mesh filename=meshes/RShoulderRoll_0.10.stl scale=0.1 0.1 0.1; visual mesh filename=meshes/RShoulderRoll_0.10.stl scale=0.1 0.1 0.1
- link RElbow: geometry collision mesh filename=meshes/RElbow_0.10.stl scale=0.1 0.1 0.1; visual mesh filename=meshes/RElbow_0.10.stl scale=0.1 0.1 0.1
- link RHipPitch: geometry collision mesh filename=meshes/RHipPitch_0.10.stl scale=0.1 0.1 0.1; visual mesh filename=meshes/RHipPitch_0.10.stl scale=0.1 0.1 0.1
- link RHipRoll: geometry collision mesh filename=meshes/RHipRoll_0.10.stl scale=0.1 0.1 0.1; visual mesh filename=meshes/RHipRoll_0.10.stl scale=0.1 0.1 0.1
- link RHipYaw: geometry collision mesh filename=meshes/RHipYaw_0.10.stl scale=0.1 0.1 0.1; visual mesh filename=meshes/RHipYaw_0.10.stl scale=0.1 0.1 0.1
- link RKnee: geometry collision mesh filename=meshes/RKnee_0.10.stl scale=0.1 0.1 0.1; visual mesh filename=meshes/RKnee_0.10.stl scale=0.1 0.1 0.1
- link RShoulder: geometry collision mesh filename=meshes/RShoulderPitch_0.10.stl scale=0.1 0.1 0.1; visual mesh filename=meshes/RShoulderPitch_0.10.stl scale=0.1 0.1 0.1
- link head: geometry collision mesh filename=meshes/Head_0.10.stl scale=0.1 0.1 0.1; visual mesh filename=meshes/Head_0.10.stl scale=0.1 0.1 0.1
- link neck: geometry collision mesh filename=meshes/Neck_0.10.stl scale=0.1 0.1 0.1; visual mesh filename=meshes/Neck_0.10.stl scale=0.1 0.1 0.1
- link torso: geometry collision mesh filename=meshes/Torso_0.10.stl scale=0.1 0.1 0.1; visual mesh filename=meshes/Torso_0.10.stl scale=0.1 0.1 0.1
Joints:
- removed joint base_link_fixedjoint
- joint LAnklePitch: origin xyz=0.0 -0.065 -0.003 rpy=0.0 0.0 0.0 -> xyz=0.0 -0.065 -0.008 rpy=0.0 0.0 0.0
- joint LAnkleRoll: origin xyz=0.0 -0.036 0.0 rpy=0.0 0.0 0.0 -> xyz=0.0 -0.035 0.0 rpy=0.0 0.0 0.0
- joint LElbowYaw: limit lower=-1.5757 upper=0.31415 effort=1.329 velocity=8.26797 -> lower=-1.5757 upper=1.5757 effort=1.329 velocity=8.26797; origin xyz=0.0745 0.0 0.0 rpy=0 -1.5757 0 -> xyz=0.075 0.0 0.0 rpy=0 -1.5757 0
- joint LHipPitch: origin xyz=0.0 -0.0426 0.0 rpy=0.0 0.0 0.0 -> xyz=0.0 -0.044 0.0 rpy=0.0 0.0 0.0
- joint LHipRoll: origin xyz=0.0 0.0 0.0905 rpy=1.5757 3.14159 0.0 -> xyz=0.0 0.0 0.09 rpy=1.5757 3.14159 0.0
- joint LHipYaw: origin xyz=0.036 -0.035 0.0 rpy=-1.5757 0.0 3.14159 -> xyz=0.035 -0.035 0.0 rpy=-1.5757 0.0 3.14159
- joint LKnee: limit lower=0.0 upper=2.05 effort=1.329 velocity=8.26797 -> lower=0.0 upper=1.5757 effort=1.329 velocity=8.26797; origin xyz=0.0 -0.065 -0.003 rpy=0.0 0.0 0.0 -> xyz=0.0 -0.06 0.0 rpy=0.0 0.0 0.0
- joint LShoulderPitch: origin xyz=0.05 0.0 0.005 rpy=0 0 0 -> xyz=0.05 0.0 0.006 rpy=0 0 0
- joint LShoulderRoll: origin xyz=0.041 0.0 0.0 rpy=0 0 0 -> xyz=0.04 0.0 0.0 rpy=0 0 0
- joint RAnklePitch: origin xyz=0.0 -0.065 -0.003 rpy=0.0 0.0 0.0 -> xyz=0.0 -0.065 -0.008 rpy=0.0 0.0 0.0
- joint RAnkleRoll: origin xyz=0.0 -0.036 0.0 rpy=0.0 0.0 0.0 -> xyz=0.0 -0.035 0.0 rpy=0.0 0.0 0.0
- joint RElbowYaw: limit lower=-0.31415 upper=1.5757 effort=1.329 velocity=8.26797 -> lower=-1.5757 upper=1.5757 effort=1.329 velocity=8.26797; origin xyz=-0.0745 0.0 0.0 rpy=0 -1.575 3.14159 -> xyz=-0.075 0.0 0.0 rpy=0 -1.575 3.14159
- joint RHipPitch: origin xyz=0.0 -0.0426 0.0 rpy=0.0 0.0 0.0 -> xyz=0.0 -0.044 0.0 rpy=0.0 0.0 0.0
- joint RHipRoll: origin xyz=0.0 0.0 0.0905 rpy=1.5757 3.14159 0.0 -> xyz=0.0 0.0 0.09 rpy=1.5757 3.14159 0.0
- joint RHipYaw: origin xyz=-0.036 -0.035 0.0 rpy=-1.5757 0.0 3.14159 -> xyz=-0.035 -0.035 0.0 rpy=-1.5757 0.0 3.14159
- joint RKnee: limit lower=0.0 upper=2.05 effort=1.329 velocity=8.26797 -> lower=0.0 upper=1.5757 effort=1.329 velocity=8.26797; origin xyz=0.0 -0.065 -0.003 rpy=0.0 0.0 0.0 -> xyz=0.0 -0.06 0.0 rpy=0.0 0.0 0.0
- joint RShoulderPitch: origin xyz=-0.05 0.0 0.005 rpy=0 0 0 -> xyz=-0.05 0.0 0.006 rpy=0 0 0
- joint RShoulderRoll: origin xyz=-0.041 0.0 0.0 rpy=0 0 0 -> xyz=-0.04 0.0 0.0 rpy=0 0 0
- joint head_to_neck: child head -> neck; origin xyz=0.0 0.0 0.0 rpy=0 0 -3.1415 -> xyz=0  0  0 rpy=0 0 0; parent neck -> head
- joint neck_to_torso: child neck -> torso; origin xyz=0.0 0.0466 0.0053 rpy=0 0 0 -> xyz=0  0  0 rpy=0 0 0; parent torso -> neck

Commit message: commit H6.urdf

File: H6.urdf (robot description, URDF)
Before this commit: robot H6_robot, 21 links, 20 joints
Joints:
- joint LAnklePitch: origin xyz=0.0 -0.065 -0.008 rpy=0.0 0.0 0.0 -> xyz=0.0 0.0 0.0 rpy=0.0 0.0 0.0
- joint LElbowYaw: axis 0 1.0 0 -> (none); origin xyz=0.075 0.0 0.0 rpy=0 -1.5757 0 -> xyz=0 0.0 0.0 rpy=0 0 0

Commit message: update URDF File

File: H6.urdf (robot description, URDF)
Before this commit: robot H6_robot, 21 links, 20 joints
Links:
- removed link LBicep
- removed link LShoulder
- removed link RBicep
- removed link RShoulder
- removed link head
- removed link neck
- removed link torso
- added link Head; collision mesh filename=meshes/Head_0.10.stl scale=0.001 0.001 0.001; visual mesh filename=meshes/Head_0.10.stl scale=0.001 0.001 0.001
- added link LShoulderPitch; collision mesh filename=meshes/LShoulderPitch_0.10.stl scale=0.001 0.001 0.001; visual mesh filename=meshes/LShoulderPitch_0.10.stl scale=0.001 0.001 0.001
- added link LShoulderRoll; collision mesh filename=meshes/LShoulderRoll_0.10.stl scale=0.001 0.001 0.001; visual mesh filename=meshes/LShoulderRoll_0.10.stl scale=0.001 0.001 0.001
- added link Neck; collision mesh filename=meshes/Neck_0.10.stl scale=0.001 0.001 0.001; visual mesh filename=meshes/Neck_0.10.stl scale=0.001 0.001 0.001
- added link RShoulderPitch; collision mesh filename=meshes/RShoulderPitch_0.10.stl scale=0.001 0.001 0.001; visual mesh filename=meshes/RShoulderPitch_0.10.stl scale=0.001 0.001 0.001
- added link RShoulderRoll; collision mesh filename=meshes/RShoulderRoll_0.10.stl scale=0.001 0.001 0.001; visual mesh filename=meshes/RShoulderRoll_0.10.stl scale=0.001 0.001 0.001
- added link Torso; collision mesh filename=meshes/Torso_0.10.stl scale=0.001 0.001 0.001; visual mesh filename=meshes/Torso_0.10.stl scale=0.001 0.001 0.001
- added link base_link
- link LAnklePitch: geometry collision mesh filename=meshes/LAnklePitch_0.10.stl scale=0.001 0.001 0.001; visual mesh filename=meshes/LAnklePitch_0.10.stl scale=0.001 0.001 0.001
- link LAnkleRoll: geometry collision mesh filename=meshes/LAnkleRoll_0.10.stl scale=0.001 0.001 0.001; visual mesh filename=meshes/LAnkleRoll_0.10.stl scale=0.001 0.001 0.001
- link LElbow: geometry collision mesh filename=meshes/LElbow_0.10.stl scale=0.001 0.001 0.001; visual mesh filename=meshes/LElbow_0.10.stl scale=0.001 0.001 0.001
- link LHipPitch: geometry collision mesh filename=meshes/LHipPitch_0.10.stl scale=0.001 0.001 0.001; visual mesh filename=meshes/LHipPitch_0.10.stl scale=0.001 0.001 0.001
- link LHipRoll: geometry collision mesh filename=meshes/LHipRoll_0.10.stl scale=0.001 0.001 0.001; visual mesh filename=meshes/LHipRoll_0.10.stl scale=0.001 0.001 0.001
- link LHipYaw: geometry collision mesh filename=meshes/LHipYaw_0.10.stl scale=0.001 0.001 0.001; visual mesh filename=meshes/LHipYaw_0.10.stl scale=0.001 0.001 0.001
- link LKnee: geometry collision mesh filename=meshes/LKnee_0.10.stl scale=0.001 0.001 0.001; visual mesh filename=meshes/LKnee_0.10.stl scale=0.001 0.001 0.001
- link RAnklePitch: geometry collision mesh filename=meshes/RAnklePitch_0.10.stl scale=0.001 0.001 0.001; visual mesh filename=meshes/RAnklePitch_0.10.stl scale=0.001 0.001 0.001
- link RAnkleRoll: geometry collision mesh filename=meshes/RAnkleRoll_0.10.stl scale=0.001 0.001 0.001; visual mesh filename=meshes/RAnkleRoll_0.10.stl scale=0.001 0.001 0.001
- link RElbow: geometry collision mesh filename=meshes/RElbow_0.10.stl scale=0.001 0.001 0.001; visual mesh filename=meshes/RElbow_0.10.stl scale=0.001 0.001 0.001
- link RHipPitch: geometry collision mesh filename=meshes/RHipPitch_0.10.stl scale=0.001 0.001 0.001; visual mesh filename=meshes/RHipPitch_0.10.stl scale=0.001 0.001 0.001
- link RHipRoll: geometry collision mesh filename=meshes/RHipRoll_0.10.stl scale=0.001 0.001 0.001; visual mesh filename=meshes/RHipRoll_0.10.stl scale=0.001 0.001 0.001
- link RHipYaw: geometry collision mesh filename=meshes/RHipYaw_0.10.stl scale=0.001 0.001 0.001; visual mesh filename=meshes/RHipYaw_0.10.stl scale=0.001 0.001 0.001
- link RKnee: geometry collision mesh filename=meshes/RKnee_0.10.stl scale=0.001 0.001 0.001; visual mesh filename=meshes/RKnee_0.10.stl scale=0.001 0.001 0.001
Joints:
- removed joint LAnklePitch
- removed joint LAnkleRoll
- removed joint LElbowYaw
- removed joint LHipPitch
- removed joint LHipRoll
- removed joint LHipYaw
- removed joint LKnee
- removed joint LShoulderPitch
- removed joint LShoulderRoll
- removed joint RAnklePitch
- removed joint RAnkleRoll
- removed joint RElbowYaw
- removed joint RHipPitch
- removed joint RHipRoll
- removed joint RHipYaw
- removed joint RKnee
- removed joint RShoulderPitch
- removed joint RShoulderRoll
- removed joint head_to_neck
- removed joint neck_to_torso
- added joint LAnklePitch_joint: type revolute, parent LKnee, child LAnklePitch, origin xyz=0.0 -0.065 -0.003 rpy=0.0 0.0 0.0, axis 1.0 0 0, limit lower=-1.0 upper=1.0 effort=1.329 velocity=8.26797
- added joint LAnkleRoll_joint: type revolute, parent LAnklePitch, child LAnkleRoll, origin xyz=0.0 -0.036 0.0 rpy=0.0 0.0 0.0, axis 0 0 1.0, limit lower=-0.85 upper=0.45 effort=1.329 velocity=8.26797
- added joint LElbow_joint: type revolute, parent LShoulderRoll, child LElbow, origin xyz=0.0745 0.0 0.0 rpy=0 0 0, axis 0 1.0 0, limit lower=-1.5757 upper=0.31415 effort=1.329 velocity=8.26797
- added joint LHipPitch_joint: type revolute, parent LHipRoll, child LHipPitch, origin xyz=0.0 -0.0426 0.0 rpy=0.0 0.0 0.0, axis 1.0 0 0, limit lower=-1.5757 upper=1.5757 effort=1.329 velocity=8.26797
- added joint LHipRoll_joint: type revolute, parent LHipYaw, child LHipRoll, origin xyz=0.0 -0.0705 0.0 rpy=0.0 0.0 0.0, axis 0 0 1.0, limit lower=-0.45 upper=1.5757 effort=1.329 velocity=8.26797
- added joint LHipYaw_joint: type revolute, parent Torso, child LHipYaw, origin xyz=0.036 -0.055 0.0 rpy=0.0 0.0 0, axis 0 1.0 0, limit lower=-1.5757 upper=1.5757 effort=1.329 velocity=8.26797
- added joint LKnee_joint: type revolute, parent LHipPitch, child LKnee, origin xyz=0.0 -0.065 -0.003 rpy=0.0 0.0 0.0, axis 1.0 0 0, limit lower=0.0 upper=2.05 effort=1.329 velocity=8.26797
- added joint LShoulderPitch_joint: type revolute, parent Torso, child LShoulderPitch, origin xyz=0.05 0.0 0.005 rpy=0 0 0, axis 1.0 0 0, limit lower=-3.1415 upper=1.0471 effort=1.329 velocity=8.26797
- added joint LShoulderRoll_joint: type revolute, parent LShoulderPitch, child LShoulderRoll, origin xyz=0.041 0.0 0.0 rpy=0 0 0, axis 0 0 1.0, limit lower=-1.5757 upper=1.5757 effort=1.329 velocity=8.26797
- added joint RAnklePitch_joint: type revolute, parent RKnee, child RAnklePitch, origin xyz=0.0 -0.065 -0.003 rpy=0.0 0.0 0.0, axis 1.0 0 0, limit lower=-1.0 upper=1.0 effort=1.329 velocity=8.26797
- added joint RAnkleRoll_joint: type revolute, parent RAnklePitch, child RAnkleRoll, origin xyz=0.0 -0.036 0.0 rpy=0.0 0.0 0.0, axis 0 0 1.0, limit lower=-0.45 upper=0.85 effort=1.329 velocity=8.26797
- added joint RElbow_joint: type revolute, parent RShoulderRoll, child RElbow, origin xyz=-0.0745 0.0 0.0 rpy=0 0 0, axis 0 1.0 0, limit lower=-0.31415 upper=1.5757 effort=1.329 velocity=8.26797
- added joint RHipPitch_joint: type revolute, parent RHipRoll, child RHipPitch, origin xyz=0.0 -0.0426 0.0 rpy=0.0 0.0 0.0, axis 1.0 0 0, limit lower=-1.5757 upper=1.5757 effort=1.329 velocity=8.26797
- added joint RHipRoll_joint: type revolute, parent RHipYaw, child RHipRoll, origin xyz=0.0 -0.0705 0.0 rpy=0.0 0.0 0.0, axis 0 0 1.0, limit lower=-1.5757 upper=0.45 effort=1.329 velocity=8.26797
- added joint RHipYaw_joint: type revolute, parent Torso, child RHipYaw, origin xyz=-0.036 -0.055 0.0 rpy=0.0 0.0 0.0, axis 0 1.0 0, limit lower=-1.5757 upper=1.5757 effort=1.329 velocity=8.26797
- added joint RKnee_joint: type revolute, parent RHipPitch, child RKnee, origin xyz=0.0 -0.065 -0.003 rpy=0.0 0.0 0.0, axis 1.0 0 0, limit lower=0.0 upper=2.05 effort=1.329 velocity=8.26797
- added joint RShoulderPitch_joint: type revolute, parent Torso, child RShoulderPitch, origin xyz=-0.05 0.0 0.005 rpy=0 0 0, axis 1.0 0 0, limit lower=-3.1415 upper=1.0471 effort=1.329 velocity=8.26797
- added joint RShoulderRoll_joint: type revolute, parent RShoulderPitch, child RShoulderRoll, origin xyz=-0.041 0.0 0.0 rpy=0 0 0, axis 0 0 1.0, limit lower=-1.5757 upper=1.5757 effort=1.329 velocity=8.26797
- added joint head_joint: type revolute, parent Neck, child Head, origin xyz=0.0 0.0 0.0 rpy=0 0 0, axis 1.0 0 0, limit lower=-0.5252 upper=0.31 effort=1.329 velocity=8.26797
- added joint neck_joint: type revolute, parent Torso, child Neck, origin xyz=0.0 0.0466 0.0053 rpy=0 0 0, axis 0 1.0 0, limit lower=-1.5757 upper=1.5757 effort=1.329 velocity=8.26797
- added joint torso_joint: type fixed, parent base_link, child Torso, origin xyz=0 0 0.35 rpy=1.5757 0 0, axis 0 0 0
